File: hardware/barrel-power-monitor.sch (KiCad schematic (older format))
At the start: 67 parts, among them J1 Barrel_Jack_Switch, J2 Barrel_Jack_Switch, J3 Conn_01x04_Male, J4 Conn_01x06_Male, J5 Conn_01x03_Male, Q1 AO3401A, Q2 2N7002, SW1 SW_Push, SW2 SW_Push, U1 STM32F030C8Tx, U2 INA139, U3 LD1117S33TR_SOT223

Commit message: v2
Parts:
- removed C1: 10n, Capacitor_SMD:C_0805_2012Metric_Pad1.18x1.45mm_HandSolder, symbol Device:C_Small
- removed D1: 4V7, Diode_SMD:D_MiniMELF, symbol Device:D_Zener
- removed JP3, JP4: SJ_NO, Jumper:SolderJumper-2_P1.3mm_Open_RoundedPad1.0x1.5mm, symbol Jumper:SolderJumper_2_Open
- removed Q2: 2N7002, Package_TO_SOT_SMD:SOT-23, symbol Transistor_FET:2N7002
- removed R2, R4: 10k 1%, Resistor_SMD:R_0402_1005Metric, symbol Device:R
- removed R3: 47k 1%, Resistor_SMD:R_0402_1005Metric, symbol Device:R
- removed R5: 2k2 1%, Resistor_SMD:R_0402_1005Metric, symbol Device:R
- removed R6: 47k, Resistor_SMD:R_0402_1005Metric, symbol Device:R_Small
- removed R7: 100, Resistor_SMD:R_0402_1005Metric, symbol Device:R_Small
- removed TP1, TP2: TestPoint, TestPoint:TestPoint_Pad_D1.5mm, symbol Connector:TestPoint
- removed U2: INA139, Package_TO_SOT_SMD:SOT-23-5, symbol Amplifier_Current:INA139
- added R10, R11: 4k7, Resistor_SMD:R_0402_1005Metric, symbol Device:R_Small
- added U2: INA219AxDCN, Package_TO_SOT_SMD:SOT-23-8, symbol Analog_ADC:INA219AxDCN
- C3: renamed from C4; value 100n 25V -> 100n; footprint Capacitor_SMD:C_0603_1608Metric -> Capacitor_SMD:C_0402_1005Metric
- renumbered C3 to C1, C5 to C4, C6 to C5, C7 to C6, C8 to C7, C9 to C8, C10 to C9, R16 to R12, R17 to R13, R18 to R14, R19 to R15, R20 to R16, R21 to R17, R8 to R2, R9 to R3, R10 to R4, R11 to R5, R12 to R6, R13 to R7, R14 to R8, R15 to R9
Connections:
- net +3V3: now also C3.1, R10.1, R11.1, U2.4 (VS); no longer R15.1
- net GND: now also D4.1 (K), U1.29 (PA8), U2.3 (GND), U2.7 (A0), U2.8 (A1)
- net VIN: now also U2.1 (IN+); no longer C3.1
- net VLOAD: now also U2.2 (IN-)
- net LED_1: now reaches U1.14 (PA4)
- net LED_1: now also R15.1
- net I2C2_SCL: now reaches U1.35 (PF6)
- net I2C2_SCL: now also R10.2, U2.5 (SCL)
- net I2C2_SDA: now reaches U1.36 (PF7)
- net I2C2_SDA: now also R11.2, U2.6 (SDA)
- net ADC_CURRENT: no longer names the net of U1.11 (PA1)
- net ADC_VOLTAGE: no longer names the net of U1.10 (PA0)
- net N_LOW_I: no longer names the net of U1.16 (PA6)
- net N_LOW_I: no longer D4.1 (K)
- net SCL renamed I2C1_SCL
- net SDA renamed I2C1_SDA
- no-connect marks 21 -> 20
Other:
- note added: "NOTE: D1 was removed,\nbut D2-D6 kept refs\nfor consistency on silk."
- note added: "PA6 used as N_LOW_I\non v1.0. Don't use."
- note removed: "10nF on ADC_CURRENT\nwas found to stabilize\nnoise from SMPS.\nWasn't necessary\non ADC_VOLTAGE.\nC1 is large to allow\nby-hand rework."
- note removed: "Keep R19 high resistance\nso MCU pin's V(OL) stays\nlow and Q1 doesn't leak."
- note removed: "Keep R6 high resistance\nso MCU pin's V(OL) stays\nlow and Q1 doesn't leak."
- note removed: "Low-current measurement mode.\nTo fully disable, close JP3.\nClose JP4 for voltage protection,\nbut might corrupt measurements\nexcept at very low current."
- note removed: "Q2 Rds(on) is not critical.\n10 ohm is fine.\nEven 100 ohm is "okay"\n(1% error in series with 10k).\nLow leakage current is important\nin low-current mode.\n50 nA is ideal (1% error at I=5 uA).\nMost datasheets don't specify this\nat low Vds."
- moved on the sheet: C3, C9, J1, J2, J5, R1, R12, R5, R6, R7
