File: hardware/barrel-power-monitor.kicad_pcb (KiCad board)
At the start: 2 copper layers, 58.4 x 33 mm, 67 parts, among them J1 Barrel_Jack_Switch, J2 Barrel_Jack_Switch, J3 Conn_01x04_Male, J4 Conn_01x06_Male, J5 Conn_01x03_Male, Q1 AO3401A, Q2 2N7002, SW1 SW_Push, SW2 SW_Push, U1 STM32F030C8Tx, U2 INA139, U3 LD1117S33TR_SOT223

Commit message: v2
Parts:
- removed the C1 at (184.8, 84.7)
- removed the C6 at (186.8, 81.5)
- removed D1: 4V7, Diode_SMD:D_MiniMELF
- removed JP3, JP4: SJ_NO, Jumper:SolderJumper-2_P1.3mm_Open_RoundedPad1.0x1.5mm
- removed Q2: 2N7002, Package_TO_SOT_SMD:SOT-23
- removed the R2 at (172.2, 78.7)
- removed the R3 at (172.2, 81.0)
- removed the R4 at (176.8, 78.1)
- removed the R5 at (177.8, 79.4)
- removed the R6 at (180.1, 84.6)
- removed the R7 at (173.1, 86.9)
- removed TP1, TP2: TestPoint, TestPoint:TestPoint_Pad_D1.5mm
- added C3: 100n, Capacitor_SMD:C_0402_1005Metric, F.Cu at (168.9, 80.8)
- added R10: 4k7, Resistor_SMD:R_0402_1005Metric, F.Cu at (182.2, 84.9)
- added R11: 4k7, Resistor_SMD:R_0402_1005Metric, F.Cu at (182.2, 83.5)
- C4: value 100n 25V -> 1u; footprint Capacitor_SMD:C_0603_1608Metric -> Capacitor_SMD:C_0402_1005Metric
- C5: value 1u -> 10n
- R1: value R100 1% -> R100 1% 2W
- U2: value INA139 -> INA219AxDCN; footprint Package_TO_SOT_SMD:SOT-23-5 -> Package_TO_SOT_SMD:SOT-23-8
- moved C4 15.8 mm to (185.7, 81.5), turned to 90 degrees
- moved U2 2.14 mm to (171.3, 79.9), turned to 0 degrees
- moved C5 1.14 mm to (186.8, 81.5)
- turned D6 to 180 degrees
- turned R17 to 180 degrees
- renumbered C3 to C1, C7 to C6, C8 to C7, C9 to C8, C10 to C9, R16 to R12, R17 to R13, R18 to R14, R19 to R15, R20 to R16, R21 to R17, R8 to R2, R9 to R3, R10 to R4, R11 to R5, R12 to R6, R13 to R7, R14 to R8, R15 to R9
Connections:
- net /SCL renamed /I2C1_SCL
- net /SDA renamed /I2C1_SDA
- C4 pad 1: /VIN -> +3.3VA
- D4 pad 1: /N_LOW_I -> GND
- R15 pad 1: +3V3 -> /LED_1
- U1 pad 10: /ADC_VOLTAGE -> Net-(U1-Pad10)
- U1 pad 11: /ADC_CURRENT -> Net-(U1-Pad11)
- U1 pad 14: Net-(U1-Pad14) -> /LED_1
- U1 pad 16: /N_LOW_I -> Net-(U1-Pad16)
- U1 pad 29: Net-(U1-Pad29) -> GND
- U1 pad 35: Net-(U1-Pad35) -> /I2C2_SCL
- U1 pad 36: Net-(U1-Pad36) -> /I2C2_SDA
- U2 pad 1: /ADC_CURRENT -> /VIN
- U2 pad 2: GND -> /VLOAD
- U2 pad 3: /VIN -> GND
- U2 pad 4: /VLOAD -> +3V3
- U2 pad 5: /VIN -> /I2C2_SCL
Routing:
- net /I2C2_SDA: track 0.00 -> 30.7 mm, vias 0 -> 2
- net /I2C2_SCL: track 0.00 -> 30.6 mm, vias 0 -> 2
- net /N_LOW_I: track 29.8 -> 0.00 mm
- net /ADC_CURRENT: track 26.2 -> 0.00 mm, vias 1 -> 0
- net /ADC_VOLTAGE: track 16.9 -> 0.00 mm
- net /LED_1: track 0.00 -> 16.2 mm
- net GND: track 21.7 -> 29.7 mm, vias 19 -> 20
- net Net-(JP3-Pad1): track 7.94 -> 0.00 mm, vias 1 -> 0
- net /VIN: track 27.3 -> 20.4 mm
- net +3V3: track 83.2 -> 89.4 mm, vias 13 -> 11
- net Net-(Q2-Pad1): track 3.33 -> 0.00 mm
- net /VLOAD: track 4.32 -> 7.36 mm
- net Net-(D1-Pad1): track 2.78 -> 0.00 mm, vias 1 -> 0
- net /LED_3: track 12.5 -> 10.9 mm
Other:
- board text added: "v2.0"
- board text removed: "Bypass"
- board text removed: "LOW-I DISABLE"
- board text removed: "Zener"
- board text removed: "v1.0"

Commit message: fix-silk-d6
Other:
- board text added: "v2.1"
- board text removed: "v2.0"
